Commit message: step 1 complete

File: Step1/r3bot.urdf (robot description, URDF)
Before this commit: robot rrbot, 5 links, 4 joints
Links:
- added link link3; visual box size=0.05 0.05 .5
Joints:
- added joint joint3: type revolute, parent link2, child link3, origin xyz=0 0.05 0.9 rpy=0 0 0, axis 0 1 0, limit lower=-1.57 upper=1.57 effort=10 velocity=1.0
- joint joint1: limit (none) -> lower=-1.57 upper=1.57 effort=10 velocity=1.0; type continuous -> revolute
- joint joint2: limit (none) -> lower=-1.57 upper=1.57 effort=10 velocity=1.0; type continuous -> revolute
- joint tool_joint: origin xyz=0 0 0.95 rpy=0 0 0 -> xyz=0 0.05 0.45 rpy=0 0 0; parent link2 -> link3
