Commit message: all of lab complete

File: Step2/m_rrbot_macro.xacro (robot description, xacro)
@@ -8,11 +8,11 @@
     <xacro:property name="height2" value="1" /> <!-- link2 -->
     <xacro:property name="axel_offset" value="0.05" /> <!-- Space between top of beam and each joint -->
-    <joint name="${prefix}_base_joint" type="fixed">
+    <joint name="${prefix}base_joint" type="fixed">
       <xacro:insert_block name="origin" />
       <parent link="${parent}" />
-      <child link="${prefix}_base_link" />
+      <child link="${prefix}base_link" />
     </joint>
     <!-- Base Link -->
-    <link name="${prefix}_base_link">
+    <link name="${prefix}base_link">
       <visual>
         <origin xyz="0 0 ${height0/2}" rpy="0 0 0"/>
@@ -23,12 +23,12 @@
       </visual>
     </link>
-    <joint name="${prefix}_joint1" type="continuous">
-      <parent link="${prefix}_base_link" />
-      <child link="${prefix}_link1" />
+    <joint name="${prefix}joint1" type="continuous">
+      <parent link="${prefix}base_link" />
+      <child link="${prefix}link1" />
       <origin xyz="0 ${width} ${height0 - axel_offset}" rpy="0 0 0" />
       <axis xyz="0 1 0" />
     </joint>
     <!-- Middle Link -->
-    <link name="${prefix}_link1">
+    <link name="${prefix}link1">
       <visual>
         <origin xyz="0 0 ${height1/2 - axel_offset}" rpy="0 0 0" />
@@ -39,12 +39,12 @@
       </visual>
     </link>
-    <joint name="${prefix}_joint2" type="continuous">
-      <parent link="${prefix}_link1" />
-      <child link="${prefix}_link2" />
+    <joint name="${prefix}joint2" type="continuous">
+      <parent link="${prefix}link1" />
+      <child link="${prefix}link2" />
       <origin xyz="0 ${width} ${height1 - axel_offset*2}" rpy="0 0 0" />
       <axis xyz="0 1 0" />
     </joint>
     <!-- Top Link -->
-    <link name="${prefix}_link2">
+    <link name="${prefix}link2">
       <visual>
         <origin xyz="0 0 ${height2/2 - axel_offset}" rpy="0 0 0" />
@@ -55,11 +55,11 @@
       </visual>
     </link>
-    <joint name="${prefix}_tool_joint" type="fixed">
+    <joint name="${prefix}tool_joint" type="fixed">
       <origin xyz="0 0 ${height2-axel_offset}" rpy="0 0 0" />
-      <parent link="${prefix}_link2" />
-      <child link="${prefix}_tool0" />
+      <parent link="${prefix}link2" />
+      <child link="${prefix}tool0" />
     </joint>
     <!-- Tool Link -->
-    <link name="${prefix}_tool0"/>
+    <link name="${prefix}tool0"/>
   </xacro:macro>
 </robot>

File: Step2/rrbot_on_table.urdf.xacro (robot description, xacro)
@@ -1,12 +1,13 @@
 <?xml version="1.0" encoding="UTF-8"?>
-<robot xmlns:xacro="http://wiki.ros.org/xacro" name="table">
+<robot xmlns:xacro="http://wiki.ros.org/xacro" name="lab_table">
+  <xacro:macro name="table" params="prefix parent *origin">
     <xacro:include filename="materials.xacro" />
     <xacro:include filename="table_macro.xacro" />
     <xacro:include filename="rrbot_macro.xacro" />
     <link name="world" />
-    <xacro:table prefix="table_" parent="world">
+    <xacro:table prefix="table" parent="world">
         <origin xyz="0 0 1" rpy="0 0 0" />
     </xacro:table>
-    <xacro:rrbot prefix="rrbot_" parent="table_top">
+    <xacro:rrbot prefix="rrbot" parent="table_top">
         <origin xyz="0 0 0" rpy="0 0 0" />
     </xacro:rrbot>
